Commit message: mounting pole working and new launch file

File: src/my_bot/description/robot.urdf.xacro (robot description, xacro)
@@ -1,4 +1,4 @@
 <?xml version="1.0"?>
-<robot xmlns:xacro="http://www.ros.org/wiki/xacro"  name="robot">
+<robot xmlns:xacro="http://www.ros.org/wiki/xacro"  name="tracker_robot">
    <xacro:include filename="robot_core.xacro"/>
    <!-- Base link -->

File: src/my_bot/description/robot_core.xacro (robot description, xacro)
@@ -3,5 +3,5 @@
 <!--Included Files-->
 <xacro:include filename="inertial_macros.xacro"/>
-<xacro:include filename="camera.xacro"/>
+<!--<xacro:include filename="camera.xacro"/> -->
 <!--Constants -->
 <xacro:property name="platform_radius" value="0.05"/>
@@ -32,4 +32,31 @@
     <link name="base_footprint">
     </link>
+<!-- Mounting Pole LINK -->
+    <joint name="mounting_pole_joint" type="fixed">
+        <parent link="base_link"/>
+        <child link="mounting_pole"/>
+        <origin xyz="0 0 0"/>
+    </joint>
+  <link name="mounting_pole">
+    <visual>
+        <origin xyz = "0 0 0"/>
+        <geometry>
+            <cylinder length="2" radius="${platform_radius}" />
+        </geometry>
+        <material name="black"/>
+    </visual>
+    <collision>
+        <origin xyz ="0 0 0"/>
+        <geometry>
+            <cylinder length="2" radius="${platform_radius}" />
+        </geometry>
+    </collision>
+    <xacro:inertial_cylinder mass = "0.1" length="2" radius="${platform_radius}">
+        <origin xyz=" 0 0 0" rpy="0 0 0"/>
+    </xacro:inertial_cylinder>
+</link>
+<gazebo reference="mounting_pole">
+    <material>Gazebo/Blue</material>
+</gazebo>
 <!-- Servo Motor Pan Platform (Bottom) -->
 <joint name="pan_platform_joint" type="continuous">
