Commit message: launch file needs fixing

File: src/my_bot/description/robot_core.xacro (robot description, xacro)
@@ -1,4 +1,12 @@
 <?xml version="1.0"?>
 <robot xmlns:xacro="http://www.ros.org/wiki/xacro" >
+<!--Included Files-->
+<xacro:include filename="inertial_macros.xacro"/>
+<xacro:include filename="camera.xacro"/>
+<!--Constants -->
+<xacro:property name="platform_radius" value="0.05"/>
+<xacro:property name="platform_length" value="0.04"/>
+<xacro:property name="tilt_platform_offset" value="0.07"/>
+<!--Material Defineitions-->
 <material name="white">
     <color rgba="1 1 1 1"/>
@@ -16,4 +24,12 @@
 <link name="base_link">
 </link>
+    <!-- BASE_FOOTPRINT LINK -->
+    <joint name="base_footprint_joint" type="fixed">
+        <parent link="base_link"/>
+        <child link="base_footprint"/>
+        <origin xyz="0 0 0" rpy="0 0 0"/>
+    </joint>
+    <link name="base_footprint">
+    </link>
 <!-- Servo Motor Pan Platform (Bottom) -->
 <joint name="pan_platform_joint" type="continuous">
@@ -26,24 +42,46 @@
     <visual>
         <geometry>
-            <cylinder length="0.04" radius="0.05" />
+            <cylinder length="${platform_length}" radius="${platform_radius}" />
         </geometry>
         <material name="blue"/>
     </visual>
+    <collision>
+        <geometry>
+            <cylinder length="${platform_length}" radius="${platform_radius}" />
+        </geometry>
+    </collision>
+    <xacro:inertial_cylinder mass = "0.1" length="${platform_length}" radius="${platform_radius}">
+        <origin xyz=" 0 0 0" rpy="0 0 0"/>
+    </xacro:inertial_cylinder>
 </link>
+<gazebo reference="pan_platform">
+    <material>Gazebo/Blue</material>
+</gazebo>
 <!-- Servo Motor Tilt Platform (Bottom) -->
 <joint name="tilt_platform_joint" type="revolute">
     <parent link="pan_platform"/>
     <child link="tilt_platform"/>
-    <origin xyz="0 0 0.07" rpy="-${pi/2} 0 0"/>
+    <origin xyz="0 0 ${tilt_platform_offset}" rpy="-${pi/2} 0 0"/>
     <axis xyz = "0 0 -1"/>
-    <limit lower = "0" upper ="${pi}" velocity = "100" effort="100"/>
+    <limit lower = "-${pi/4}" upper ="${pi/2}" velocity = "100" effort="100"/>
 </joint>
 <link name="tilt_platform">
     <visual>
         <geometry>
-            <cylinder length="0.04" radius="0.05" />
+            <cylinder length="${platform_length}" radius="${platform_radius}" />
         </geometry>
         <material name="orange"/>
     </visual>
+    <collision>
+        <geometry>
+            <cylinder length="${platform_length}" radius="${platform_radius}" />
+        </geometry>
+    </collision>
+    <xacro:inertial_cylinder mass = "0.1" length="${platform_length}" radius="${platform_radius}">
+        <origin xyz=" 0 0 0" rpy="0 0 0"/>
+    </xacro:inertial_cylinder>
 </link>
+<gazebo reference="tilt_platform">
+    <material>Gazebo/Orange</material>
+</gazebo>
 </robot>

Commit message: mounting pole included loads into gazebo

File: src/my_bot/description/robot_core.xacro (robot description, xacro)
@@ -3,9 +3,10 @@
 <!--Included Files-->
 <xacro:include filename="inertial_macros.xacro"/>
-<!--<xacro:include filename="camera.xacro"/> -->
+<xacro:include filename="camera.xacro"/>
 <!--Constants -->
 <xacro:property name="platform_radius" value="0.05"/>
 <xacro:property name="platform_length" value="0.04"/>
 <xacro:property name="tilt_platform_offset" value="0.07"/>
+<xacro:property name="pan_platform_offset" value="1.02"/>
 <!--Material Defineitions-->
 <material name="white">
@@ -36,5 +37,5 @@
         <parent link="base_link"/>
         <child link="mounting_pole"/>
-        <origin xyz="0 0 0"/>
+        <origin xyz="0 0 1"/>
     </joint>
   <link name="mounting_pole">
@@ -44,8 +45,8 @@
             <cylinder length="2" radius="${platform_radius}" />
         </geometry>
-        <material name="black"/>
+        <material name="white"/>
     </visual>
     <collision>
-        <origin xyz ="0 0 0"/>
+        <origin xyz ="0 0 1"/>
         <geometry>
             <cylinder length="2" radius="${platform_radius}" />
@@ -53,15 +54,15 @@
     </collision>
     <xacro:inertial_cylinder mass = "0.1" length="2" radius="${platform_radius}">
-        <origin xyz=" 0 0 0" rpy="0 0 0"/>
+        <origin xyz=" 0 0 -1" rpy="0 0 0"/>
     </xacro:inertial_cylinder>
 </link>
 <gazebo reference="mounting_pole">
-    <material>Gazebo/Blue</material>
+    <material>Gazebo/White</material>
 </gazebo>
 <!-- Servo Motor Pan Platform (Bottom) -->
 <joint name="pan_platform_joint" type="continuous">
-    <parent link="base_link"/>
+    <parent link="mounting_pole"/>
     <child link="pan_platform"/>
-    <origin xyz="0 0 0" rpy="0 0 0"/>
+    <origin xyz="0 0 ${pan_platform_offset}" rpy="0 0 0"/>
     <axis xyz="0 0 1"/>
 </joint>
