Commit message: errors but fixing the controller issues

File: src/my_bot/description/ros2_control.xacro (robot description, xacro)
@@ -6,14 +6,29 @@
         </hardware>
         <joint name="pan_platform_joint">
-            <command_interface name="position">
-            </command_interface>
+            <command_interface name="position" /> <!--These command and state interface must match yaml controller-->
             <state_interface name="position"/>
         </joint>
         <joint name="tilt_platform_joint">
-            <command_interface name="position">
-            </command_interface>
+            <command_interface name="position" />
             <state_interface name="position"/>
         </joint>
     </ros2_control>
+ <!-- might not need these-->
+    <gazebo reference="pan_platform">
+        <material>Gazebo/Blue</material>
+        <plugin filename="gz-sim-joint-state-publisher-system" name="gz::sim::systems::JointStatePublisher">
+            <topic>joint_states</topic>
+            <joint_name>pan_platform_joint</joint_name>
+            <joint_name>tilt_platform_joint</joint_name>
+        </plugin>
+    </gazebo>
+    <gazebo reference="tilt_mount_pole">
+        <material>Gazebo/White</material>
+        <plugin filename="gz-sim-joint-state-publisher-system" name="gz::sim::systems::JointStatePublisher">
+            <topic>joint_states</topic>
+            <joint_name>pan_platform_joint</joint_name>
+            <joint_name>tilt_platform_joint</joint_name>
+        </plugin>
+    </gazebo>
     <gazebo>
         <plugin name="gz_ros2_control::GazeboSimROS2ControlPlugin" filename="libgz_ros2_control-system.so">
