Commit message: trying to update the controllers

File: src/my_bot/description/camera.xacro (robot description, xacro)
@@ -28,5 +28,5 @@
         <parent link="camera_link"/>
         <child link="camera_link_optical"/>
-        <origin xyz="0 0 0" rpy="${-pi/2} 0 ${-pi/2}"/>
+        <origin xyz="0 0 0" rpy="${-pi/2} 0 0"/>
     </joint>
     <link name="camera_link_optical"></link>

File: src/my_bot/description/robot.urdf.xacro (robot description, xacro)
@@ -2,4 +2,5 @@
 <robot xmlns:xacro="http://www.ros.org/wiki/xacro"  name="tracker_robot">
    <xacro:include filename="robot_core.xacro"/>
+   <xacro:include filename="ros2_control.xacro"/>
    <!-- Base link -->
 </robot>

File: src/my_bot/description/robot_core.xacro (robot description, xacro)
@@ -7,6 +7,10 @@
 <xacro:property name="platform_radius" value="0.05"/>
 <xacro:property name="platform_length" value="0.04"/>
-<xacro:property name="tilt_platform_offset" value="0.07"/>
+<xacro:property name="tilt_platform_offset" value="0.125"/>
 <xacro:property name="pan_platform_offset" value="1.02"/>
+<xacro:property name="tilt_mount_pole_radius" value="0.01"/>
+<xacro:property name="tilt_mount_pole_offset" value="0.03"/>
+<xacro:property name="tilt_mount_pole_length" value="0.1"/>
+<xacro:property name="mount_pole_radius" value="0.03"/>
 <!--Material Defineitions-->
 <material name="white">
@@ -43,5 +47,5 @@
         <origin xyz = "0 0 0"/>
         <geometry>
-            <cylinder length="2" radius="${platform_radius}" />
+            <cylinder length="2" radius="${mount_pole_radius}" />
         </geometry>
         <material name="white"/>
@@ -50,8 +54,8 @@
         <origin xyz ="0 0 1"/>
         <geometry>
-            <cylinder length="2" radius="${platform_radius}" />
+            <cylinder length="2" radius="${mount_pole_radius}" />
         </geometry>
     </collision>
-    <xacro:inertial_cylinder mass = "0.1" length="2" radius="${platform_radius}">
+    <xacro:inertial_cylinder mass = "0.1" length="2" radius="${mount_pole_radius}">
         <origin xyz=" 0 0 -1" rpy="0 0 0"/>
     </xacro:inertial_cylinder>
@@ -86,7 +90,34 @@
     <material>Gazebo/Blue</material>
 </gazebo>
+<!-- Tilt Mount Pole LINK -->
+    <joint name="tilt_mount_pole_joint" type="fixed">
+        <parent link="pan_platform"/>
+        <child link="tilt_mount_pole"/>
+        <origin xyz="0 0 ${tilt_mount_pole_offset}"/>
+    </joint>
+  <link name="tilt_mount_pole">
+    <visual>
+        <origin xyz = "0 0 ${tilt_mount_pole_offset}"/>
+        <geometry>
+            <cylinder length="${tilt_mount_pole_length}" radius="${tilt_mount_pole_radius}" />
+        </geometry>
+        <material name="white"/>
+    </visual>
+    <collision>
+        <origin xyz ="0 0 ${tilt_mount_pole_offset}"/>
+        <geometry>
+            <cylinder length="${tilt_mount_pole_length}" radius="${tilt_mount_pole_radius}" />
+        </geometry>
+    </collision>
+    <xacro:inertial_cylinder mass = "0.1" length="${tilt_mount_pole_length}" radius="${tilt_mount_pole_radius}">
+        <origin xyz=" 0 0 ${tilt_mount_pole_offset}" rpy="0 0 0"/>
+    </xacro:inertial_cylinder>
+</link>
+<gazebo reference="tilt_mount_pole">
+    <material>Gazebo/White</material>
+</gazebo>
 <!-- Servo Motor Tilt Platform (Bottom) -->
 <joint name="tilt_platform_joint" type="revolute">
-    <parent link="pan_platform"/>
+    <parent link="tilt_mount_pole"/>
     <child link="tilt_platform"/>
     <origin xyz="0 0 ${tilt_platform_offset}" rpy="-${pi/2} 0 0"/>

File: src/my_bot/description/ros2_control.xacro (robot description, xacro)
@@ -1,61 +1,27 @@
 <?xml version="1.0"?>
 <robot xmlns:xacro="http://www.ros.org/wiki/xacro">
-    <xacro:unless value="$(arg sim_mode)">
-        <ros2_control name="RealRobot" type="system">
-            <hardware>
-                <plugin>diffdrive_arduino/DiffDriveArduinoHardware</plugin>
-                <param name="left_wheel_name">left_wheel_joint</param>
-                <param name="right_wheel_name">right_wheel_joint</param>
-                <param name="loop_rate">30</param>
-                <param name="device">/dev/ttyUSB0</param>
-                <param name="baud_rate">57600</param>
-                <param name="timeout_ms">1000</param>
-                <param name="enc_counts_per_rev">3436</param>
-            </hardware>
-            <joint name="left_wheel_joint">
-                <command_interface name="velocity">
-                    <param name="min">-10</param>
-                    <param name="max">10</param>
-                </command_interface>
-                <state_interface name="position"/>
-                <state_interface name="velocity"/>
-            </joint>
-            <joint name="right_wheel_joint">
-                <command_interface name="velocity">
-                    <param name="min">-10</param>
-                    <param name="max">10</param>
-                </command_interface>
-                <state_interface name="position"/>
-                <state_interface name="velocity"/>
-            </joint>
-        </ros2_control>
-    </xacro:unless>
-    <xacro:if value="$(arg sim_mode)">
-        <ros2_control name="GazeboSystem" type="system">
-            <hardware>
-                <plugin>gz_ros2_control/GazeboSimSystem</plugin>
-            </hardware>
-            <joint name="left_wheel_joint">
-                <command_interface name="velocity">
-                    <param name="min">-10</param>
-                    <param name="max">10</param>
-                </command_interface>
-                <state_interface name="velocity"/>
-                <state_interface name="position"/>
-            </joint>
-            <joint name="right_wheel_joint">
-                <command_interface name="velocity">
-                    <param name="min">-10</param>
-                    <param name="max">10</param>
-                </command_interface>
-                <state_interface name="velocity"/>
-                <state_interface name="position"/>
-            </joint>
-        </ros2_control>
-    </xacro:if>
+    <ros2_control name="GazeboSystem" type="system">
+        <hardware>
+            <plugin>gz_ros2_control/GazeboSimSystem</plugin>
+        </hardware>
+        <joint name="pan_platform_joint">
+            <command_interface name="position">
+            <param name="min">-100</param>
+            <param name="max">100</param>
+            </command_interface>
+            <state_interface name="position"/>
+        </joint>
+        <joint name="tilt_platform_joint">
+            <command_interface name="position">
+            <param name="min">-100</param>
+            <param name="max">100</param>
+            </command_interface>
+            <state_interface name="position"/>
+        </joint>
+    </ros2_control>
     <gazebo>
         <plugin name="gz_ros2_control::GazeboSimROS2ControlPlugin" filename="libgz_ros2_control-system.so">
-            <parameters>$(find articubot_one)/config/my_controllers.yaml</parameters>
-            <parameters>$(find articubot_one)/config/gaz_ros2_ctl_use_sim.yaml</parameters>
+            <parameters>$(find my_bot)/config/my_controllers.yaml</parameters>
+            <parameters>$(find my_bot)/config/gaz_ros2_ctl_use_sim.yaml</parameters>
         </plugin>
     </gazebo>

Commit message: contorrler problms

File: src/my_bot/description/camera.xacro (robot description, xacro)
@@ -28,5 +28,5 @@
         <parent link="camera_link"/>
         <child link="camera_link_optical"/>
-        <origin xyz="0 0 0" rpy="${-pi/2} 0 0"/>
+        <origin xyz="0 0 0" rpy="${-pi/2} 0 ${-pi/2}"/>
     </joint>
     <link name="camera_link_optical"></link>

File: src/my_bot/description/robot_core.xacro (robot description, xacro)
@@ -65,9 +65,10 @@
 </gazebo>
 <!-- Servo Motor Pan Platform (Bottom) -->
-<joint name="pan_platform_joint" type="continuous">
+<joint name="pan_platform_joint" type="revolute">
     <parent link="mounting_pole"/>
     <child link="pan_platform"/>
     <origin xyz="0 0 ${pan_platform_offset}" rpy="0 0 0"/>
     <axis xyz="0 0 1"/>
+   <!-- <limit lower = "0" upper ="6.28" velocity = "100" effort="100"/>    -->
 </joint>
 <link name="pan_platform">
@@ -123,5 +124,5 @@
     <origin xyz="0 0 ${tilt_platform_offset}" rpy="-${pi/2} 0 0"/>
     <axis xyz = "0 0 -1"/>
-    <limit lower = "-${pi/4}" upper ="${pi/2}" velocity = "100" effort="100"/>
+    <!--<limit lower = "-0.78" upper ="1.57" velocity = "100" effort="100"/> -->
 </joint>
 <link name="tilt_platform">

File: src/my_bot/description/ros2_control.xacro (robot description, xacro)
@@ -1,4 +1,5 @@
 <?xml version="1.0"?>
 <robot xmlns:xacro="http://www.ros.org/wiki/xacro">
+<!--can delete the Sim from line below to make like articulated-->
     <ros2_control name="GazeboSystem" type="system">
         <hardware>
@@ -6,29 +7,26 @@
         </hardware>
         <joint name="pan_platform_joint">
-            <command_interface name="position" /> <!--These command and state interface must match yaml controller-->
-            <state_interface name="position"/>
+            <command_interface name="position" > <!--These command and state interface must match yaml-->
+                <param name="min">"0"</param>
+                <param name="max">6.28</param>
+            </command_interface>
+            <state_interface name="position">
+                <param name="initial_value">0</param>
+            </state_interface>
+            <state_interface name="velocity"/>
+            <state_interface name="effort"/>
         </joint>
         <joint name="tilt_platform_joint">
-            <command_interface name="position" />
-            <state_interface name="position"/>
+            <command_interface name="position">
+                <param name="min">"-0.78"</param>
+                <param name="max">1.57</param>
+            </command_interface>
+            <state_interface name="position">
+                <param name="initial_value">0</param>
+            </state_interface>
+            <state_interface name="velocity"/>
+            <state_interface name="effort"/>
         </joint>
     </ros2_control>
- <!-- might not need these-->
-    <gazebo reference="pan_platform">
-        <material>Gazebo/Blue</material>
-        <plugin filename="gz-sim-joint-state-publisher-system" name="gz::sim::systems::JointStatePublisher">
-            <topic>joint_states</topic>
-            <joint_name>pan_platform_joint</joint_name>
-            <joint_name>tilt_platform_joint</joint_name>
-        </plugin>
-    </gazebo>
-    <gazebo reference="tilt_mount_pole">
-        <material>Gazebo/White</material>
-        <plugin filename="gz-sim-joint-state-publisher-system" name="gz::sim::systems::JointStatePublisher">
-            <topic>joint_states</topic>
-            <joint_name>pan_platform_joint</joint_name>
-            <joint_name>tilt_platform_joint</joint_name>
-        </plugin>
-    </gazebo>
     <gazebo>
         <plugin name="gz_ros2_control::GazeboSimROS2ControlPlugin" filename="libgz_ros2_control-system.so">
@@ -38,2 +36,4 @@
     </gazebo>
 </robot>
+<!--
+<plugin name="gz_ros2_control::GazeboSimROS2ControlPlugin" filename="gz_ros2_control-system"></plugin> -->
